File: KiCad/BIT90_26/BIT90_26_Processor.kicad_sch (KiCad schematic)
At the start: 39 parts, among them J11 Clock Test Points, SW1 [RST], SW68 ROM BANK SELECT, U10 Z80, U11 74LS74, U17 6264, U18 74LS32, U19 74LS04, U20 74LS107, U5 74LS05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

Commit message: Minor corrections & footprints assigned
PCB layout started
Parts:
- removed unit 1 of U5
- added unit 1 of U14
- C5, C6, C7: footprint (none) -> Capacitor_THT:C_Disc_D3.4mm_W2.1mm_P2.50mm
- C8, C9: footprint (none) -> Capacitor_THT:CP_Radial_D6.3mm_P2.50mm
- D2, D3, D4: footprint (none) -> Diode_THT:D_DO-35_SOD27_P7.62mm_Horizontal
- J11: footprint (none) -> Connector_PinHeader_2.54mm:PinHeader_1x05_P2.54mm_Vertical
- R11, R12, R13, R14, R15, R17, R18, R19, R20, R21, R22, R23, R24, R30, R31: footprint (none) -> Resistor_THT:R_Axial_DIN0207_L6.3mm_D2.5mm_P7.62mm_Horizontal
- R16: value R -> 10KΩ; footprint (none) -> Resistor_THT:R_Axial_DIN0207_L6.3mm_D2.5mm_P7.62mm_Horizontal
- SW1: footprint (none) -> Clueless_Engineer:SW_Gateron_LowProfile_THT
- SW68: footprint (none) -> Button_Switch_THT:SW_DIP_SPSTx02_Slide_9.78x7.26mm_W7.62mm_P2.54mm
- U10: renamed from U19; footprint (none) -> Package_DIP:DIP-14_W7.62mm
- U11: renamed from U6; footprint (none) -> Package_DIP:DIP-16_W7.62mm
- U14: renamed from U5; footprint (none) -> Package_DIP:DIP-14_W7.62mm
- U15: renamed from U20; footprint (none) -> Package_DIP:DIP-14_W7.62mm
- U7: renamed from U11; footprint (none) -> Package_DIP:DIP-14_W7.62mm
- U8: renamed from U18; footprint (none) -> Package_DIP:DIP-14_W7.62mm
- Y1: footprint (none) -> Crystal:Crystal_HC49-U_Vertical
- renumbered U17 to U1, U7 to U2, U8 to U3, U9 to U4, U10 to U5
Connections:
- net +5V: now also R16.2, U11.6 (E3); no longer R16.1
- net ~{DISM}: now also R16.1; no longer R16.2, U11.6 (E3)
- net ~{RFSH}: now also U14.1
- net ~{EXT_RST}: now reaches C8.1, R23.1, SW1.2
- net ~{INT}: now reaches R18.2, U14.6, U5.16 (~{INT})
- net at U11.5 (E2): now also U14.2
- net RES renamed RESET
Other:
- moved on the sheet: R16, R23
