File: KiCad/BIT90_26/BIT90_26_Controllers.kicad_sch (KiCad schematic)
At the start: 11 parts, among them U19 74LS04, U2 74LS244, U22 74LS00, U23 74LS00, U3 74LS244, U4 74LS138, U5 74LS05

Commit message: Minor corrections & footprints assigned
PCB layout started
Parts:
- removed U5: 74LS05, symbol 74xx:74LS05
- added U14: 74LS05, Package_DIP:DIP-14_W7.62mm, symbol 74xx:74LS05
- R7, R8: footprint (none) -> Resistor_THT:R_Axial_DIN0207_L6.3mm_D2.5mm_P7.62mm_Horizontal
- RN2: value R_Network08 -> 10KΩ
- U10: renamed from U19; footprint (none) -> Package_DIP:DIP-14_W7.62mm
- U12: renamed from U23; footprint (none) -> Package_DIP:DIP-14_W7.62mm
- U13: renamed from U4; footprint (none) -> Package_DIP:DIP-16_W7.62mm
- U33: renamed from U3; footprint (none) -> Package_DIP:DIP-20_W7.62mm
- U34: renamed from U2; footprint (none) -> Package_DIP:DIP-20_W7.62mm
- U9: renamed from U22; footprint (none) -> Package_DIP:DIP-14_W7.62mm
Connections:
- net at U13.7 (O7): now also U14.9
- net at U12.13, U12.5: now also U14.8
- net ~{DISM} renamed ~{DISIO}

Commit message: PCB layout started
Connections:
- net CTRL1_PIN2: now also RN2.5 (R4); no longer RN2.4 (R3)
- net CTRL1_PIN3: now also RN2.7 (R6); no longer RN2.5 (R4)
- net CTRL1_PIN6: now also RN2.6 (R5); no longer RN2.8 (R7)
- net CTRL1_PIN7: now also RN2.8 (R7); no longer RN2.7 (R6)
- net CTRL2_PIN3: now also RN3.6 (R5); no longer RN3.5 (R4)
- net CTRL2_PIN6: now also RN3.5 (R4); no longer RN3.8 (R7)
- net at U34.11 (I0b): now also RN3.8 (R7); no longer RN3.6 (R5)
- net at U33.11 (I0b): now also RN2.9 (R8); no longer RN2.6 (R5)
- net at U33.17 (I3b): now also RN2.4 (R3); no longer RN2.9 (R8)
