File: KiCad/BIT90_26/BIT90_26_Keyboard_Interfaces.kicad_sch (KiCad schematic)
At the start: 86 parts, among them J1 Cartridge, J2 Expansion, J3 Joystick 1, J4 Joystick 2, J5 TAPE DUMP, J6 TAPE LOAD, J7 AUDIO OUT, SW10 CARAT, SW11 8, SW12 4, SW13 BS, SW14 DEL, SW15 2, SW16 6, SW17 ZERO, SW18 P, SW19 Y, SW2 MINUS, SW20 W, SW21 ], SW22 UP, SW23 ESC, SW24 R, SW25 I, SW26 [, SW27 U, SW28 E, SW29 RUBOUT, SW3 7, SW30 RIGHT, SW31 Q, SW32 T, SW33 O, SW34 SEMICOLON, SW35 H, SW36 S, SW37 AT, SW38 FWDSLASH, SW39 CAPS/LOWER, SW4 3, SW40 F, SW41 K, SW42 COLON, SW43 J, SW44 D, SW45 CR, SW46 PERIOD, SW47 A, SW48 G, SW49 L, SW5 BACKSLASH, SW50 N, SW51 V, SW52 X, SW53 M, SW54 COMMA, SW55 Z, SW56 C, SW57 B, SW58 R_SHIFT, SW59 R_SHIFT, SW6 INS, SW60 BIT, SW61 BASIC, SW62 LEFT, SW63 DOWN, SW64 CTRL, SW65 SPACE, SW66 FCTN, SW7 1, SW8 5, SW9 6, U12 74LS145, U13 74LS174, U14 74LS244, U15 LM393

Commit message: Minor corrections & footprints assigned
PCB layout started
Parts:
- added J12: Expansion2, Connector_PinHeader_2.54mm:PinHeader_2x30_P2.54mm_Vertical, symbol Connector_Generic:Conn_02x30_Counter_Clockwise
- C10: footprint (none) -> Capacitor_THT:C_Disc_D3.4mm_W2.1mm_P2.50mm
- C11: value 2.2nF (222) -> 0nF; footprint (none) -> Capacitor_THT:C_Disc_D3.4mm_W2.1mm_P2.50mm
- D5, D6: footprint (none) -> Diode_THT:D_DO-35_SOD27_P7.62mm_Horizontal
- J1: footprint (none) -> Clueless_Engineer:CONN30_2x15_DRXN_SUL
- J2: footprint (none) -> Clueless_Engineer:BIT90 Expansion
- J3, J4: footprint (none) -> Connector_Dsub:DSUB-9_Pins_Horizontal_P2.77x2.84mm_EdgePinOffset7.70mm_Housed_MountingHolesOffset9.12mm
- J5, J6, J7: footprint (none) -> Clueless_Engineer:SJ335083ATR
- R25, R26, R27, R29: footprint (none) -> Resistor_THT:R_Axial_DIN0207_L6.3mm_D2.5mm_P7.62mm_Horizontal
- R28: value 56KΩ -> 0KΩ; footprint (none) -> Resistor_THT:R_Axial_DIN0207_L6.3mm_D2.5mm_P7.62mm_Horizontal
- SW10, SW11, SW12, SW13, SW14, SW15, SW16, SW17, SW18, SW19, SW2, SW20, SW21, SW22, SW23, SW24, SW25, SW26, SW27, SW28, SW29, SW3, SW30, SW31, SW32, SW33, SW34, SW35, SW36, SW37, SW38, SW39, SW4, SW40, SW41, SW42, SW43, SW44, SW45, SW46, SW47, SW48, SW49, SW5, SW50, SW51, SW52, SW53, SW54, SW55, SW56, SW57, SW58, SW59, SW6, SW60, SW61, SW62, SW63, SW64, SW65, SW66, SW7, SW8, SW9: footprint (none) -> Clueless_Engineer:SW_Gateron_LowProfile_THT
- U25: renamed from U15; footprint (none) -> Package_DIP:DIP-8_W7.62mm
- U30: renamed from U12; footprint (none) -> Package_DIP:DIP-16_W7.62mm
- U31: renamed from U14; footprint (none) -> Package_DIP:DIP-20_W7.62mm
- U32: renamed from U13; footprint (none) -> Package_DIP:DIP-16_W7.62mm
Connections:
- net +12V: now also J12.57 (Pin_57)
- net +5V: now also J12.58 (Pin_58), J12.59 (Pin_59)
- net -5V: now also J12.60 (Pin_60)
- net A0: now also J12.47 (Pin_47)
- net A1: now also J12.18 (Pin_18)
- net A10: now also J12.28 (Pin_28)
- net A11: now also J12.37 (Pin_37)
- net A12: now also J12.38 (Pin_38)
- net A13: now also J12.22 (Pin_22)
- net A14: now also J12.4 (Pin_4)
- net A15: now also J12.43 (Pin_43)
- net A2: now also J12.20 (Pin_20)
- net A3: now also J12.44 (Pin_44)
- net A4: now also J12.21 (Pin_21)
- net A5: now also J12.23 (Pin_23)
- net A6: now also J12.24 (Pin_24)
- net A7: now also J12.25 (Pin_25)
- net A8: now also J12.26 (Pin_26)
- net A9: now also J12.27 (Pin_27)
- net AUDIO_OUT: now also J12.56 (Pin_56)
- net AUDΦ: now also J12.35 (Pin_35)
- net CPUΦ: now also J12.45 (Pin_45)
- net D0: now also J12.14 (Pin_14)
- net D1: now also J12.12 (Pin_12)
- net D2: now also J12.46 (Pin_46)
- net D3: now also J12.3 (Pin_3)
- net D4: now also J12.19 (Pin_19)
- net D5: now also J12.48 (Pin_48)
- net D6: now also J12.17 (Pin_17)
- net D7: now also J12.16 (Pin_16)
- net GND: now also J12.1 (Pin_1), J12.2 (Pin_2)
- net INT: now also J12.10 (Pin_10)
- net RΦ: now also J12.40 (Pin_40)
- net ~{BUSAK}: now also J12.52 (Pin_52)
- net ~{BUSRQ}: now also J12.11 (Pin_11)
- net ~{DISM}: now also J12.29 (Pin_29)
- net ~{HALT}: now also J12.7 (Pin_7)
- net ~{INT}: now also J12.51 (Pin_51)
- net ~{IORQ}: now also J12.55 (Pin_55)
- net ~{M1}: now also J12.15 (Pin_15)
- net ~{MERQ}: now also J12.54 (Pin_54)
- net ~{MS4}_(40): now also J12.5 (Pin_5)
- net ~{NMI}: now also J12.9 (Pin_9)
- net ~{RD}: now also J12.53 (Pin_53)
- net ~{RFSH}: now also J12.49 (Pin_49)
- net ~{RST}: now also J12.13 (Pin_13)
- net ~{RST}/SY: now also J12.39 (Pin_39)
- net ~{WAIT}: now also J12.50 (Pin_50)
- net ~{WR}: now also J12.8 (Pin_8)
- net DISIO renamed ~{DISIO}
- net ~{DISIO}: now also J12.30 (Pin_30)
- net EXTAD renamed EXT_AUD
- net EXT_AUD: now also J12.31 (Pin_31)
- net EXTV: no longer names the net of J2.33 (Pin_33)
- net EXTVE: no longer names the net of J2.32 (Pin_32)
- net RES renamed RESET
- net RESET: now also J12.36 (Pin_36)
- net ~{RS1} renamed ~{EXT_RST}
- net ~{EXT_RST}: now also J12.34 (Pin_34)
- no-connect marks 8 -> 15
Other:
- moved on the sheet: J1, J2

Commit message: PCB layout started
Parts:
- SW2: value MINUS -> UNDERSCORE
- SW58: value R_SHIFT -> L_SHIFT
- SW9: value 6 -> 9
Connections:
- net GND: now also J3.0 (SH), J4.0 (SH)
- net KI_{2}: now also RN1.5 (R4); no longer RN1.4 (R3)
- net KI_{3}: now also RN1.7 (R6); no longer RN1.5 (R4)
- net KI_{4}: now also RN1.9 (R8); no longer RN1.6 (R5)
- net KI_{5}: now also RN1.8 (R7); no longer RN1.7 (R6)
- net KI_{6}: now also RN1.6 (R5); no longer RN1.8 (R7)
- net KI_{7}: now also RN1.4 (R3); no longer RN1.9 (R8)
- net EXP32: now reaches J12.32 (Pin_32)
- net EXP32: now also J2.32 (Pin_32)
- net EXP33: now reaches J12.33 (Pin_33)
- net EXP33: now also J2.33 (Pin_33)
- net EXP41: now reaches J12.41 (Pin_41)
- net EXP41: now also J2.41 (Pin_41)
- net EXP42: now reaches J12.42 (Pin_42)
- net EXP42: now also J2.42 (Pin_42)
- net EXP6: now reaches J12.6 (Pin_6)
- net EXP6: now also J2.6 (Pin_6)
- no-connect marks 15 -> 5
