File: KiCad/BIT90_26/BIT90_26_Power.kicad_sch (KiCad schematic)
At the start: 36 parts, among them J10 +5V In, J8 Mean Well PSU, J9 +5V In, SW67 ON/OFF, U11 74LS74, U15 LM393, U18 74LS32, U19 74LS04, U20 74LS107, U22 74LS00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

Commit message: Minor corrections & footprints assigned
PCB layout started
Parts:
- added C33, C34, C35: 10µF/16V, Capacitor_THT:CP_Radial_D6.3mm_P2.50mm, symbol Device:C_Polarized
- C12, C13, C14, C15, C16, C17, C18, C19, C20, C21, C22, C23, C24, C25, C26, C27, C28, C29, C3, C30, C31, C32: footprint (none) -> Capacitor_THT:C_Disc_D3.4mm_W2.1mm_P2.50mm
- C2: footprint (none) -> Capacitor_THT:CP_Radial_D6.3mm_P2.50mm
- F1: footprint (none) -> Fuse:Fuseholder_Clip-5x20mm_Littelfuse_111_Inline_P20.00x5.00mm_D1.05mm_Horizontal
- J10: value +5V In -> +5V In (2.1mm); footprint (none) -> Connector_BarrelJack:BarrelJack_Horizontal
- J8: footprint (none) -> Clueless_Engineer:SDF80J
- J9: value +5V In -> +5V In (USB); footprint (none) -> Connector_USB:USB_B_Lumberg_2411_02_Horizontal
- SW67: footprint (none) -> Clueless_Engineer:SW_400MSP1R6BLKM6QE
- U10: renamed from U19; footprint (none) -> Package_DIP:DIP-14_W7.62mm
- U12: renamed from U23; footprint (none) -> Package_DIP:DIP-14_W7.62mm
- U14: renamed from U5; footprint (none) -> Package_DIP:DIP-14_W7.62mm
- U15: renamed from U20; footprint (none) -> Package_DIP:DIP-14_W7.62mm
- U25: renamed from U15; footprint (none) -> Package_DIP:DIP-8_W7.62mm
- U7: renamed from U11; footprint (none) -> Package_DIP:DIP-14_W7.62mm
- U8: renamed from U18; footprint (none) -> Package_DIP:DIP-14_W7.62mm
- U9: renamed from U22; footprint (none) -> Package_DIP:DIP-14_W7.62mm
Connections:
- net +5V: now also C33.1, C34.1, C35.1
- net GND: now also C33.2, C34.2, C35.2
Other:
- note added: "For expansion/cartridge"
- note added: "Orignally for TMS9929"
- moved on the sheet: C12, C13, C14, C15, C16, C17, C18, C19, C2, C20, C21, C22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

Commit message: PCB layout started
Parts:
- added D7: POWER, LED_THT:LED_D5.0mm, symbol Device:LED
- added R32: R, Resistor_THT:R_Axial_DIN0207_L6.3mm_D2.5mm_P7.62mm_Horizontal, symbol Device:R
- J8: value Mean Well PSU -> Mean Well GP25A13A-R1B
Connections:
- net +5V: now also R32.1
- net GND: now also SW67.S (SPT), D7.1 (K)
- new net: D7.2 (A), R32.2
Changed lines of the file:
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@@
 	)
 	(junction
+		(at 368.3 36.83)
+		(diameter 0)
+		(color 0 0 0 0)
+	)
+	(junction
 		(at 171.45 102.87)
 		(diameter 0)
@@
 	(wire
 		(pts
+			(xy 378.46 46.99) (xy 368.3 46.99)
+		)
+		(stroke
+			(width 0)
+			(type default)
+		)
+	)
+	(wire
+		(pts
 			(xy 93.98 102.87) (xy 113.03 102.87)
 		)
@@
 	(wire
 		(pts
+			(xy 368.3 38.1) (xy 368.3 36.83)
+		)
+		(stroke
+			(width 0)
+			(type default)
+		)
+	)
+	(wire
+		(pts
 			(xy 373.38 36.83) (xy 368.3 36.83)
 		)
@@
 	(wire
 		(pts
+			(xy 368.3 46.99) (xy 368.3 45.72)
+		)
+		(stroke
+			(width 0)
+			(type default)
+		)
+	)
+	(wire
+		(pts
 			(xy 113.03 95.25) (xy 133.35 95.25)
 		)
@@
 	(wire
 		(pts
+			(xy 388.62 46.99) (xy 386.08 46.99)
+		)
+		(stroke
+			(width 0)
+			(type default)
+		)
+	)
+	(wire
+		(pts
 			(xy 358.14 36.83) (xy 351.79 36.83)
 		)
@@
 	(global_label "GND"
 		(shape input)
+		(at 360.68 41.91 270)
+		(fields_autoplaced yes)
+		(effects
+			(font
+				(size 1.27 1.27)
+			)
+			(justify right)
+		)
+		(property "Intersheetrefs" "${INTERSHEET_REFS}"
+			(at 360.68 48.7657 90)
+			(effects
+				(font
+					(size 1.27 1.27)
+				)
+				(justify right)
+				(hide yes)
+			)
+		)
+	)
+	(global_label "GND"
+		(shape input)
 		(at 27.94 234.95 180)
 		(fields_autoplaced yes)
@@
 		)
 	)
+	(global_label "GND"
+		(shape input)
+		(at 388.62 46.99 0)
+		(fields_autoplaced yes)
+		(effects
+			(font
+				(size 1.27 1.27)
+			)
+			(justify left)
+		)
+		(property "Intersheetrefs" "${INTERSHEET_REFS}"
+			(at 395.4757 46.99 0)
+			(effects
+				(font
+					(size 1.27 1.27)
+				)
+				(justify left)
+				(hide yes)
+			)
+		)
+	)
 	(global_label "+5V"
 		(shape input)
@@
 		(fields_autoplaced yes)
 		(property "Reference" "J8"
-			(at 314.9601 83.82 0)
+			(at 314.96 83.82 0)
 			(effects
 				(font
@@
 			)
 		)
-		(property "Value" "Mean Well PSU"
-			(at 314.9601 86.36 0)
+		(property "Value" "Mean Well GP25A13A-R1B"
+			(at 314.96 86.36 0)
 			(effects
 				(font
@@
 		)
 		(property "Footprint" "Clueless_Engineer:SW_400MSP1R6BLKM6QE"
-			(at 363.22 36.83 0)
+			(at 363.22 26.67 0)
 			(effects
 				(font
@@
 		)
 		(property "Description" "Single Pole Single Throw (SPST) switch"
-			(at 363.22 36.83 0)
+			(at 363.22 29.21 0)
 			(effects
 				(font
@@
 		(pin "1"
 		)
+		(pin "S"
+		)
 		(instances
 			(project "BIT90_26"
@@
 	)
 	(symbol
+		(lib_id "Device:LED")
+		(at 382.27 46.99 180)
+		(unit 1)
+		(exclude_from_sim no)
+		(in_bom yes)
+		(on_board yes)
+		(dnp no)
+		(fields_autoplaced yes)
+		(property "Reference" "D7"
+			(at 383.8575 39.37 0)
+			(effects
+				(font
+					(size 1.27 1.27)
+				)
+			)
+		)
+		(property "Value" "POWER"
+			(at 383.8575 41.91 0)
+			(effects
+				(font
+					(size 1.27 1.27)
+				)
+			)
+		)
+		(property "Footprint" "LED_THT:LED_D5.0mm"
+			(at 382.27 46.99 0)
+			(effects
+				(font
+					(size 1.27 1.27)
+				)
+				(hide yes)
+			)
+		)
+		(property "Datasheet" "~"
+			(at 382.27 46.99 0)
+			(effects
+				(font
+					(size 1.27 1.27)
+				)
+				(hide yes)
+			)
+		)
+		(property "Description" "Light emitting diode"
+			(at 382.27 46.99 0)
+			(effects
+				(font
+					(size 1.27 1.27)
+				)
+				(hide yes)
+			)
+		)
+		(property "Sim.Pins" "1=K 2=A"
+			(at 382.27 46.99 0)
+			(effects
+				(font
+					(size 1.27 1.27)
+				)
+				(hide yes)
+			)
+		)
+		(pin "2"
+		)
+		(pin "1"
+		)
+		(instances
+			(project "BIT90_26"
+				(path "/d65498c3-6385-4920-ac0f-4c76daf90780/4eb1b27c-0de4-437c-bec4-8709ba05b3a7"
+					(reference "D7")
+					(unit 1)
+				)
+			)
+		)
+	)
+	(symbol
 		(lib_id "74xx:74LS32")
 		(at 35.56 252.73 0)
@@
 					(unit 1)
 				)
+			)
+		)
+	)
+	(symbol
+		(lib_id "Device:R")
+		(at 368.3 41.91 0)
+		(unit 1)
+		(exclude_from_sim no)
+		(in_bom yes)
+		(on_board yes)
+		(dnp no)
+		(fields_autoplaced yes)
+		(property "Reference" "R32"
+			(at 370.84 40.6399 0)
+			(effects
+				(font
+					(size 1.27 1.27)
+				)
+				(justify left)
+			)
+		)
+		(property "Value" "R"
+			(at 370.84 43.1799 0)
+			(effects
+				(font
+					(size 1.27 1.27)
+				)
+				(justify left)
+			)
+		)
+		(property "Footprint" "Resistor_THT:R_Axial_DIN0207_L6.3mm_D2.5mm_P7.62mm_Horizontal"
+			(at 366.522 41.91 90)
+			(effects
+				(font
+					(size 1.27 1.27)
+				)
+				(hide yes)
+			)
+		)
+		(property "Datasheet" "~"
+			(at 368.3 41.91 0)
+			(effects
+				(font
+					(size 1.27 1.27)
+				)
+				(hide yes)
+			)
+		)
+		(property "Description" "Resistor"
+			(at 368.3 41.91 0)
+			(effects
+				(font
+					(size 1.27 1.27)
+				)
+				(hide yes)
+			)
+		)
+		(pin "2"
+		)
+		(pin "1"
+		)
+		(instances
+			(project "BIT90_26"
+				(path "/d65498c3-6385-4920-ac0f-4c76daf90780/4eb1b27c-0de4-437c-bec4-8709ba05b3a7"
+					(reference "R32")
+					(unit 1)
+				)
