File: KiCad/BIT90_Original/BIT90_Keyboard.kicad_sch (KiCad schematic)
At the start: 73 parts, among them SW1 MINUS, SW10 8, SW11 4, SW12 BS, SW13 DEL, SW14 2, SW15 6, SW16 ZERO, SW17 P, SW18 Y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

Commit message: Minor corrections
Parts:
- SW66: value R_SHIFT -> L_SHIFT
- SW8: value 6 -> 9
