File: KiCad/BIT90_Original/BIT90_Video_Encoder_PAL.kicad_sch (KiCad schematic)
At the start: 7 parts, among them Q5 2N2222

Commit message: Completed original schematic redraw
Well, didn't finish the Video Encoder (PAL) sheet as I'm not going to use any of it in the new design.
Moved the audio output from that sheet to the Joystick/Audio/Tape out sheet where the sound generator is.
Parts:
- removed C60: C, symbol Device:C
- removed Q5: 2N2222, symbol Simulation_SPICE:NPN
- removed R64: 22KΩ, symbol Device:R
- removed R65: 10KΩ, symbol Device:R
- removed R66: 6.8KΩ, symbol Device:R
- removed R67: 330Ω, symbol Device:R
- removed R7: 56KΩ, symbol Device:R
- added C52, C54, C58: 100nF, symbol Device:C
- added C55: 33pF, symbol Device:C
- added C56: 47pF, symbol Device:C
- added C58: 10µF/16V, symbol Device:C_Polarized
- added C?: ??, symbol Device:C_Polarized
- added L1: 39µH, symbol Device:L
- added L2: 15µH, symbol Device:L
- added Q1: 2N2907, symbol Simulation_SPICE:PNP
- added Q2: 2N2222, symbol Simulation_SPICE:NPN
- added R53: 3.3KΩ, symbol Device:R
- added R54: 2,7KΩ, symbol Device:R
- added R55: 120KΩ, symbol Device:R
- added R57: 100Ω, symbol Device:R
- added R58: 27KΩ, symbol Device:R
- added R60: 1.7KΩ, symbol Device:R
- added R61: 330Ω, symbol Device:R
- added U26, U29: CD4066BE, Package_DIP:DIP-14_W7.62mm, symbol Analog_Switch:CD4066BE
- added U27: LM1889, Package_DIP:DIP-18_W7.62mm, symbol Clueless_Engineer:LM1889
- added U28: CD4013, Package_DIP:DIP-14_W7.62mm, symbol Clueless_Engineer:CD4013
Connections:
- net +12V: now also Q1.3 (E), Q2.1 (C)
- net GND: now also C55.2, C58.2, R54.2, R55.2, R57.2, R61.2, U28.10 (RESET), U28.8 (SET)
- new net: C58.1, R60.2, R61.1, U26.11
- new net: C?.1, Q1.2 (B), R55.1
- new net: Q1.1 (C), R54.1
- new net: R58.2, U28.11 (CLOCK)
- new net: U28.12 (~{Q}), U28.9 (DATA)
- new net: C56.1, L2.2, R58.1, U26.12, U26.13, U26.5, U26.6
- new net: C56.2, L2.1, Q2.3 (E)
- new net: L1.1, R53.2
- new net: C55.1, L1.2, Q2.2 (B)
- new net: C54.2, R53.1, U26.8
- new net +5V: R60.1
- new net B-Y: C52.1
- new net B-Y_INPUT: C52.2, U26.4, U27.4 (B-Y_INPUT)
- new net CHROMA_BIAS: U26.2, U26.3, U27.3 (CHROMA_BIAS)
- new net R-Y: C58.1
- new net R-Y_INPUT: C58.2, U26.1, U27.2 (R-Y_INPUT)
- new net Y: C54.1, C?.2, R57.1
