File: KiCad/BIT90_26_Prototype/BIT90_26_Processor.kicad_sch (KiCad schematic)
At the start: 39 parts, among them J11 Clock Test Points, SW1 [RST], SW68 ROM BANK SELECT, U1 6264, U10 74LS04, U11 74LS138, U14 74LS05, U15 74LS107, U2 27C256, U3 27C256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

Commit message: Moved initial design to Prototype folder
Parts:
- D2, D3, D4: footprint Diode_THT:D_DO-35_SOD27_P7.62mm_Horizontal -> Clueless_Engineer:D_DO-35_SOD27_P7.62mm_Horizontal
Connections:
- net +5V: now also U15.10 (~{R}), U15.13 (~{R})
- no-connect marks 4 -> 2

Commit message: Added more signal analysis to schematic
Would be nice to reduce the amount of glue logic
Changed lines of the file:
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@@
 		)
 	)
-	(text_box "CPUΦ = CPU clock\nVDPΦ = video clock\nAUDΦ = audio clock (called EXTΦ on BIT90)\nRΦ = current-limited CPU clock to expansion"
+	(text_box "~{MO} & ~{BA1} BEHAVIOUR\nA13 = H\nA14 = H\nA15 = H\n\n~{MO} ASSERTS WHEN A3 = L\n~{BA1} ASSERTS WHEN A3 = H\n\nY1 IS STROBE"
+		(exclude_from_sim no)
+		(at 176.53 50.8 0)
+		(size 30.48 20.32)
+		(margins 0.9525 0.9525 0.9525 0.9525)
+		(stroke
+			(width 0)
+			(type solid)
+		)
+		(fill
+			(type none)
+		)
+		(effects
+			(font
+				(size 1.27 1.27)
+			)
+			(justify left top)
+		)
+	)
+	(text_box "CPUΦ = CPU clock (3.57MHz)\nVDPΦ = video clock (10.73864MHz)\nAUDΦ = audio clock (called EXTΦ on BIT90)\nRΦ = current-limited CPU clock to expansion"
 		(exclude_from_sim no)
 		(at 154.94 251.46 0)
