File: KiCad/BIT90_26_Prototype/BIT90_26_Prototype.kicad_pcb (KiCad board)
At the start: 2 copper layers, 182 parts, among them J1 Cartridge, J10 +5V In (2.1mm), J11 Clock Test Points, J12 Expansion2, J2 Expansion, J3 Joystick 1, J4 Joystick 2, J5 TAPE DUMP, J6 TAPE LOAD, J7 AUDIO OUT, J8 Mean Well GP25A13A-R1B, J9 +5V In (USB), Q1 2N2222, SW1 [RST], SW10 CARAT, SW11 8, SW12 4, SW13 BS, SW14 DEL, SW15 2, SW16 6, SW17 ZERO, SW18 P, SW19 Y, SW2 UNDERSCORE, SW20 W, SW21 ], SW22 UP, SW23 ESC, SW24 R, SW25 I, SW26 [, SW27 U, SW28 E, SW29 RUBOUT, SW3 7, SW30 RIGHT, SW31 Q, SW32 T, SW33 O, SW34 SEMICOLON, SW35 H, SW36 S, SW37 AT, SW38 FWDSLASH, SW39 CAPS/LOWER, SW4 3, SW40 F, SW41 K, SW42 COLON, SW43 J, SW44 D, SW45 CR, SW46 PERIOD, SW47 A, SW48 G, SW49 L, SW5 BACKSLASH, SW50 N, SW51 V, SW52 X, SW53 M, SW54 COMMA, SW55 Z, SW56 C, SW57 B, SW58 L_SHIFT, SW59 R_SHIFT, SW6 INS, SW60 BIT, SW61 BASIC, SW62 LEFT, SW63 DOWN, SW64 CTRL, SW65 SPACE, SW66 FCTN, SW67 ON/OFF, SW68 ROM BANK SELECT, SW7 1, SW8 5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

Commit message: Moved initial design to Prototype folder
Parts:
- removed C11: 0nF, Capacitor_THT:C_Disc_D3.4mm_W2.1mm_P2.50mm
- removed R28: 0KΩ, Resistor_THT:R_Axial_DIN0207_L6.3mm_D2.5mm_P7.62mm_Horizontal
- added J13: HDMI For Pico9918, Clueless_Engineer:Pico9918_HDMI_Board, F.Cu at (154.2, 51.3)
- D1, D2, D3, D4, D5, D6: footprint Diode_THT:D_DO-35_SOD27_P7.62mm_Horizontal -> Clueless_Engineer:D_DO-35_SOD27_P7.62mm_Horizontal
- moved R27 327.5 mm to (245.9, 81.8), turned to -90 degrees
- moved R29 320.8 mm to (242.7, 89.4), turned to 90 degrees
- moved Y1 288.6 mm to (-113.9, 75.4)
- moved D2 279.2 mm to (211.0, 111.6), turned to -90 degrees
- moved D4 259.0 mm to (190.7, 118.0), turned to 90 degrees
- moved D3 255.7 mm to (186.9, 110.3), turned to -90 degrees
- moved C17 251.1 mm to (-108.4, 116.7)
- moved C18 251.1 mm to (-107.2, 56.4)
- moved C19 251.1 mm to (-104.6, 68.5)
- moved C20 251.1 mm to (-104.6, 80.5)
- moved C27 251.1 mm to (-104.6, 92.6)
- moved C28 251.1 mm to (-104.6, 104.7)
- moved R9 251.1 mm to (-98.9, 111.6)
- moved U10 251.1 mm to (-101.4, 73.5)
- moved U6 251.1 mm to (-104.0, 121.8)
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Connections:
- R27 pad 2: Net-(C11-Pad1) -> GND
- R29 pad 1: Net-(C11-Pad1) -> GND
- U15 pad 10: unconnected-(U15B-~{R}-Pad10) -> +5V
- U15 pad 13: unconnected-(U15A-~{R}-Pad13) -> +5V
- U32 pad 15: Net-(U32-Q5) -> GND
Routing:
- net KI_{3}: track 154.0 -> 247.6 mm
- net D1: track 71.0 -> 138.5 mm
- net D0: track 71.0 -> 137.6 mm
- net D2: track 67.5 -> 126.3 mm
- net A12: track 67.6 -> 124.8 mm
- net A0: track 67.5 -> 122.9 mm
- net A1: track 71.1 -> 123.5 mm
- net A2: track 71.1 -> 121.9 mm
- net A4: track 71.0 -> 119.3 mm
- net D7: track 71.0 -> 118.4 mm
- net A5: track 71.0 -> 117.3 mm
- net A6: track 71.0 -> 114.2 mm
- net A7: track 71.1 -> 113.0 mm
- net SOUND_OUT: track 0.00 -> 41.5 mm
- net D6: track 71.0 -> 109.7 mm
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Other:
- board text added: "PROTOTYPE"

Commit message: Added more signal analysis to schematic
Would be nice to reduce the amount of glue logic
Parts:
- removed C2, C35: 10µF/16V, Capacitor_THT:CP_Radial_D6.3mm_P2.50mm
- added H1: MountingHole, MountingHole:MountingHole_3.2mm_M3, F.Cu at (480.2, 254.6)
- added H2: MountingHole, MountingHole:MountingHole_3.2mm_M3, F.Cu at (480.2, 151.6)
- added H3: MountingHole, MountingHole:MountingHole_3.2mm_M3, F.Cu at (162.2, 151.6)
- added H4: MountingHole, MountingHole:MountingHole_3.2mm_M3, F.Cu at (480.2, 344.6)
- added H5: MountingHole, MountingHole:MountingHole_3.2mm_M3, F.Cu at (162.2, 254.6)
- added H6: MountingHole, MountingHole:MountingHole_3.2mm_M3, F.Cu at (162.2, 344.6)
- C1: value 100nF -> 1nF (102)
- moved U9 555.1 mm to (437.3, 219.4), turned to 0 degrees
- moved Y1 554.5 mm to (427.1, 197.0)
- moved U10 547.4 mm to (426.2, 219.2), turned to 0 degrees
- moved C28 547.4 mm to (431.3, 216.1), turned to 180 degrees
- moved C20 533.7 mm to (408.5, 227.4)
- moved C17 514.4 mm to (401.2, 186.7)
- moved U13 499.8 mm to (415.5, 219.2), turned to 0 degrees
- moved C19 481.5 mm to (355.1, 211.6), turned to 0 degrees
- moved U6 447.5 mm to (327.2, 241.6), turned to 180 degrees
- moved C6 446.7 mm to (438.6, 203.5)
- moved C7 446.7 mm to (438.6, 206.7)
- moved R11 446.7 mm to (415.8, 203.5)
- moved R12 446.7 mm to (426.0, 203.5)
- moved C5 446.7 mm to (423.5, 206.7), turned to 0 degrees
- moved C18 424.3 mm to (295.7, 189.5), turned to 0 degrees
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Routing:
- net +12V: track 7.62 -> 184.3 mm
- net -5V: track 7.62 -> 172.4 mm, vias 0 -> 1
- net +5V: track 71.4 -> 217.5 mm
- net GND: track 149.5 -> 286.2 mm
- net KI_{7}: track 167.8 -> 263.9 mm, vias 0 -> 2
- net AUDIO_OUT: track 11.4 -> 98.9 mm
- net KO_{5}: track 231.5 -> 318.1 mm
- net CTRL_COMMON_2: track 0.00 -> 85.6 mm
- net KI_{4}: track 135.1 -> 207.8 mm, vias 0 -> 1
- net D7: track 118.4 -> 186.9 mm
- net D3: track 103.2 -> 167.8 mm
- net KO_{3}: track 315.2 -> 374.1 mm
- net AUDΦ: track 7.62 -> 66.5 mm
- net D4: track 101.2 -> 159.6 mm
- net ~{WAIT}: track 7.62 -> 58.6 mm
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- added copper zone on B.Cu, net GND
Other:
- board outline added: 325 x 209 mm
